Commit message: Xacro modular code improvements

File: urdf/gazebo_tags/gazebo_plugins.xacro (robot description, xacro)
@@ -7,7 +7,6 @@
             <wheel_separation>0.15</wheel_separation>
             <wheel_radius>0.068</wheel_radius>
-            <!--Best to use prefixes for frame ID's ('robotname/odom' for example) and to set the prefix on the RVIZ config too-->
-            <frame_id>tribot/odom</frame_id>
-            <child_frame_id>tribot/base_footprint</child_frame_id>
+            <frame_id>${robot_name}/odom</frame_id>
+            <child_frame_id>${robot_name}/base_footprint</child_frame_id>
         </plugin>
     </gazebo>

File: urdf/modules/tribot_chassis_and_wheels.xacro (robot description, xacro)
@@ -21,5 +21,5 @@
       <origin xyz="0 -0.001 0" rpy="0 -0 0"/>
       <geometry>
-        <mesh filename="package://tribot_description/assets/chassis.stl"/>
+        <mesh filename="package://${package_name}/assets/chassis.stl"/>
       </geometry>
       <material name="chassis_material">
@@ -30,5 +30,5 @@
       <origin xyz="0 -0.001 0" rpy="0 -0 0"/>
       <geometry>
-        <mesh filename="package://tribot_description/assets/chassis.stl"/>
+        <mesh filename="package://${package_name}/assets/chassis.stl"/>
       </geometry>
     </collision>
@@ -45,5 +45,5 @@
       <origin xyz="0 0 0.035" rpy="-1.5708 -0 0"/>
       <geometry>
-        <mesh filename="package://tribot_description/assets/driven_wheel.stl"/>
+        <mesh filename="package://${package_name}/assets/driven_wheel.stl"/>
       </geometry>
       <material name="driven_wheel_material">
@@ -54,5 +54,5 @@
       <origin xyz="0 0 0.035" rpy="-1.5708 -0 0"/>
       <geometry>
-        <mesh filename="package://tribot_description/assets/driven_wheel.stl"/>
+        <mesh filename="package://${package_name}/assets/driven_wheel.stl"/>
       </geometry>
     </collision>
@@ -77,5 +77,5 @@
       <origin xyz="0 0 0.035" rpy="-1.5708 -0 0"/>
       <geometry>
-        <mesh filename="package://tribot_description/assets/driven_wheel.stl"/>
+        <mesh filename="package://${package_name}/assets/driven_wheel.stl"/>
       </geometry>
       <material name="driven_wheel_2_material">
@@ -86,5 +86,5 @@
       <origin xyz="0 0 0.035" rpy="-1.5708 -0 0"/>
       <geometry>
-        <mesh filename="package://tribot_description/assets/driven_wheel.stl"/>
+        <mesh filename="package://${package_name}/assets/driven_wheel.stl"/>
       </geometry>
     </collision>
@@ -109,5 +109,5 @@
       <origin xyz="-0.0075 -0.0075 0.005" rpy="3.14159 -0 0"/>
       <geometry>
-        <mesh filename="package://tribot_description/assets/caster_frame.stl"/>
+        <mesh filename="package://${package_name}/assets/caster_frame.stl"/>
       </geometry>
       <material name="caster_frame_material">
@@ -118,5 +118,5 @@
       <origin xyz="-0.0075 -0.0075 0.005" rpy="3.14159 -0 0"/>
       <geometry>
-        <mesh filename="package://tribot_description/assets/caster_frame.stl"/>
+        <mesh filename="package://${package_name}/assets/caster_frame.stl"/>
       </geometry>
     </collision>
@@ -141,5 +141,5 @@
       <origin xyz="0 0 0.0085" rpy="1.5708 -0 0"/>
       <geometry>
-        <mesh filename="package://tribot_description/assets/caster_wheel.stl"/>
+        <mesh filename="package://${package_name}/assets/caster_wheel.stl"/>
       </geometry>
       <material name="caster_wheel_material">
@@ -150,5 +150,5 @@
       <origin xyz="0 0 0.0085" rpy="1.5708 -0 0"/>
       <geometry>
-        <mesh filename="package://tribot_description/assets/caster_wheel.stl"/>
+        <mesh filename="package://${package_name}/assets/caster_wheel.stl"/>
       </geometry>
     </collision>

File: urdf/robot.urdf.xacro (robot description, xacro)
@@ -1,4 +1,5 @@
 <?xml version="1.0" ?>
 <robot name="tribot" xmlns:xacro="http://www.ros.org/wiki/xacro">
+    <xacro:include filename="xacro_properties/xacro_properties.xacro" />
     <xacro:include filename="modules/tribot_chassis_and_wheels.xacro" />
     <xacro:include filename="gazebo_tags/gazebo_plugins.xacro" />
